Commit message: Port drix_description from ROS 1 (catkin) to ROS 2 (ament_cmake)
- Convert package.xml from catkin to ament_cmake, add joint/robot state publisher deps
- Convert CMakeLists.txt to ament_cmake pattern (matching ben_description)
- Update URDF with placeholder box geometry, inertial properties, and DriX-specific
  propulsion (prop + rudder joint) for Gazebo simulation compatibility
- Add GPS and IMU sensor frames
- Convert ROS 1 XML launch files to ROS 2 Python launch files (load, publish_state, display)
- Add ament environment hooks for GZ_SIM_RESOURCE_PATH
- Add RViz config for URDF visualization

Closes rolker/drix_description#2

Co-Authored-By: Claude Opus 4.6 <noreply@anthropic.com>

File: urdf/drix_mesh.xacro (robot description, xacro)
@@ -1,15 +1,44 @@
 <?xml version="1.0"?>
 <robot xmlns:xacro="http://ros.org/wiki/xacro" name="drix">
-  <xacro:arg name="drixNumber" default="1"/>
-  <xacro:arg name="namespace" default="drix_$(arg drixNumber)"/>
+  <xacro:arg name="namespace" default="drix"/>
   <xacro:property name="namespace" value="$(arg namespace)" scope="global" />
+  <!-- DriX hull: ~7.7m long, ~2.0m wide, ~2.5m tall
+       Mass: 2200 kg (measured weight with water in gondola)
+       Using placeholder box geometry until meshes are available. -->
+  <xacro:property name="hull_length" value="7.7" />
+  <xacro:property name="hull_width" value="2.0" />
+  <xacro:property name="hull_height" value="1.5" />
+  <xacro:property name="hull_mass" value="2200.0" />
   <link name="${namespace}/base_link">
+    <inertial>
+      <mass value="${hull_mass}" />
+      <origin xyz="0 0 0" rpy="0 0 0" />
+      <inertia
+        ixx="${hull_mass * (hull_width * hull_width + hull_height * hull_height) / 12.0}"
+        ixy="0" ixz="0"
+        iyy="${hull_mass * (hull_length * hull_length + hull_height * hull_height) / 12.0}"
+        iyz="0"
+        izz="${hull_mass * (hull_length * hull_length + hull_width * hull_width) / 12.0}" />
+    </inertial>
     <visual>
-        <geometry>
-            <mesh filename="package://drix_description/models/meshes/drix.dae"/>
-        </geometry>
+      <geometry>
+        <box size="${hull_length} ${hull_width} ${hull_height}" />
+      </geometry>
+      <material name="drix_hull">
+        <color rgba="1.0 0.55 0.0 1.0" />
+      </material>
     </visual>
+    <collision>
+      <geometry>
+        <box size="${hull_length} ${hull_width} ${hull_height}" />
+      </geometry>
+    </collision>
   </link>
+  <!-- EK80 sonar (hull-mounted, pointing down) -->
   <link name="${namespace}/ek80">
+    <inertial>
+      <mass value="2.0" />
+      <inertia ixx="0.001" ixy="0" ixz="0" iyy="0.001" iyz="0" izz="0.001" />
+    </inertial>
     <visual>
       <geometry>
@@ -18,45 +47,107 @@
       <origin rpy="0 1.57075 0" xyz="-0.0376 0 0"/>
     </visual>
-  </link>
-  <joint name="${namespace}/base_to_ek80" type="fixed">
-      <parent link="${namespace}/base_link"/>
-      <child link="${namespace}/ek80"/>
-      <!-- <origin rpy="0 1.57075 0" xyz="-0.728 -0.131 -0.134 " /> -->
-      <origin rpy="3.14 0 0" xyz="-0.728 -0.131 -0.134 " />
-  </joint>
-  <link name="sonar_vcs">
-    <visual>
+    <collision>
       <geometry>
         <cylinder length="0.0752" radius="0.06"/>
       </geometry>
       <origin rpy="0 1.57075 0" xyz="-0.0376 0 0"/>
+    </collision>
+  </link>
+  <joint name="${namespace}/base_to_ek80" type="fixed">
+    <parent link="${namespace}/base_link"/>
+    <child link="${namespace}/ek80"/>
+    <origin rpy="3.14 0 0" xyz="-0.728 -0.131 -0.134" />
+  </joint>
+  <!-- GPS antenna -->
+  <link name="${namespace}/gps">
+    <inertial>
+      <mass value="0.5" />
+      <inertia ixx="0.0001" ixy="0" ixz="0" iyy="0.0001" iyz="0" izz="0.0001" />
+    </inertial>
+    <visual>
+      <geometry>
+        <cylinder length="0.05" radius="0.08" />
+      </geometry>
     </visual>
+    <collision>
+      <geometry>
+        <cylinder length="0.05" radius="0.08" />
+      </geometry>
+    </collision>
   </link>
-  <link name="${namespace}/base_link_north_up">
+  <joint name="${namespace}/base_to_gps" type="fixed">
+    <parent link="${namespace}/base_link"/>
+    <child link="${namespace}/gps"/>
+    <origin xyz="1.0 0 1.2" rpy="0 0 0" />
+  </joint>
+  <!-- IMU / heading sensor -->
+  <link name="${namespace}/imu">
+    <inertial>
+      <mass value="1.0" />
+      <inertia ixx="0.001" ixy="0" ixz="0" iyy="0.001" iyz="0" izz="0.001" />
+    </inertial>
+  </link>
+  <joint name="${namespace}/base_to_imu" type="fixed">
+    <parent link="${namespace}/base_link"/>
+    <child link="${namespace}/imu"/>
+    <origin xyz="0 0 0" rpy="0 0 0" />
+  </joint>
+  <!-- Rudder: DriX uses prop + rudder steering
+       Rudder distance from CG: 3.4m (from asv_sim config)
+       Max rudder angle: 30 degrees -->
+  <link name="${namespace}/rudder">
+    <inertial>
+      <mass value="10.0" />
+      <inertia ixx="0.01" ixy="0" ixz="0" iyy="0.01" iyz="0" izz="0.01" />
+    </inertial>
     <visual>
-        <geometry>
-            <sphere radius="0.01"/>
-        </geometry>
+      <geometry>
+        <box size="0.3 0.02 0.4" />
+      </geometry>
+      <material name="rudder_material">
+        <color rgba="0.5 0.5 0.5 1.0" />
+      </material>
     </visual>
+    <collision>
+      <geometry>
+        <box size="0.3 0.02 0.4" />
+      </geometry>
+    </collision>
   </link>
-  <joint name="${namespace}/base_north_up_to_base" type="floating">
-    <parent link="${namespace}/base_link_north_up"/>
-    <child link="${namespace}/base_link"/>
+  <joint name="${namespace}/rudder_joint" type="revolute">
+    <parent link="${namespace}/base_link"/>
+    <child link="${namespace}/rudder"/>
+    <origin xyz="-3.4 0 -0.5" rpy="0 0 0" />
+    <axis xyz="0 0 1" />
+    <limit lower="${-30.0 * 3.14159 / 180.0}" upper="${30.0 * 3.14159 / 180.0}"
+           effort="100" velocity="1.57" />
   </joint>
-  <link name="${namespace}/base_link_level">
+  <!-- Propeller -->
+  <link name="${namespace}/propeller">
+    <inertial>
+      <mass value="5.0" />
+      <inertia ixx="0.01" ixy="0" ixz="0" iyy="0.01" iyz="0" izz="0.02" />
+    </inertial>
     <visual>
-        <geometry>
-            <sphere radius="0.01"/>
-        </geometry>
+      <geometry>
+        <cylinder length="0.05" radius="0.15" />
+      </geometry>
+      <origin rpy="0 1.5708 0" xyz="0 0 0" />
+      <material name="propeller_material">
+        <color rgba="0.3 0.3 0.3 1.0" />
+      </material>
     </visual>
+    <collision>
+      <geometry>
+        <cylinder length="0.05" radius="0.15" />
+      </geometry>
+      <origin rpy="0 1.5708 0" xyz="0 0 0" />
+    </collision>
   </link>
-  <joint name="${namespace}/base_north_up_to_base_level" type="floating">
-    <parent link="${namespace}/base_link_north_up"/>
-    <child link="${namespace}/base_link_level"/>
-  </joint>
-  <joint name="${namespace}/base_to_sonar_vcs" type="fixed">
-    <parent link="${namespace}/base_link_level"/>
-    <child link="sonar_vcs"/>
-    <origin rpy="3.14 0 0" xyz="-0.586 0.080 -0.149 " />
+  <joint name="${namespace}/propeller_joint" type="continuous">
+    <parent link="${namespace}/base_link"/>
+    <child link="${namespace}/propeller"/>
+    <origin xyz="-3.6 0 -0.5" rpy="0 0 0" />
+    <axis xyz="1 0 0" />
   </joint>
 </robot>
